File: hardware/control-unit-pcb/control-unit-pcb.sch (KiCad schematic (older format))
At the start: 6 parts, among them P1 Digital, P2 Analog, P3 CONN_01X01, P4 CONN_01X01, P5 CONN_01X01, P6 CONN_01X01

Commit message: Assign some footprints
Parts:
- removed P1: Digital, Socket_Arduino_Nano:Socket_Strip_Arduino_1x15, symbol Connector_Generic:Conn_01x15
- removed P2: Analog, Socket_Arduino_Nano:Socket_Strip_Arduino_1x15, symbol Connector_Generic:Conn_01x15
- removed P3, P4, P5, P6: CONN_01X01, Socket_Arduino_Nano:1pin_Nano, symbol Connector_Generic:Conn_01x01
- added A1: Arduino_Nano_v3.x, Module:Arduino_Nano, symbol MCU_Module:Arduino_Nano_v3.x
- added C1: 1uF, Capacitor_THT:CP_Radial_D4.0mm_P1.50mm, symbol Device:CP
- added C2: 100nF, Capacitor_SMD:C_1206_3216Metric_Pad1.42x1.75mm_HandSolder, symbol Device:C
- added C3, C4: 100nF, symbol Device:C
- added H1, H2, H3, H4: MountingHole, MountingHole:MountingHole_3mm, symbol Mechanical:MountingHole
- added H5: MountingHole, MountingHole:MountingHole_8.4mm_M8, symbol Mechanical:MountingHole
- added J1, J2: Conn_01x04_Male, Connector_PinSocket_2.54mm:PinSocket_1x04_P2.54mm_Vertical, symbol Connector:Conn_01x04_Male
- added J3, J4: Screw_Terminal_01x03, TerminalBlock:TerminalBlock_Altech_AK300-3_P5.00mm, symbol Connector:Screw_Terminal_01x03
- added J5: Screw_Terminal_01x02, TerminalBlock:TerminalBlock_Altech_AK300-2_P5.00mm, symbol Connector:Screw_Terminal_01x02
- added J6: Conn_02x10_Row_Letter_Last, TerminalBlock_PTR:TerminalBlock_PTR_AKZ3191_10KD-2x10_2.54x5.00, symbol Connector_Generic:Conn_02x10_Row_Letter_Last
- added J7: Conn_01x02_Male, Connector_JST:JST_XH_B2B-XH-A_1x02_P2.50mm_Vertical, symbol Connector:Conn_01x02_Male
- added R1: 2k2, symbol Device:R
- added R2: 1k2, symbol Device:R
- added R3, R4, R5, R6, R7: R, symbol Device:R
- added R8: 2M, symbol Device:R
- added R9: 10M, symbol Device:R
Connections:
- net labels added: BTN_1, BTN_2, BTN_3, LED_BL, LED_BR, LED_FL, LED_FR, RX, TX, VCC
- net labels removed: +3.3V, 0(Rx), 1(Tx), 10(**/SS), 11(**/MOSI), 12(MISO), 13(SCK), 2, 3(**), 4, 5(**), 6(**), 7, 8, 9(**), A0, A1, A2, A3, A4, A5, A6, A7, AREF, Reset, Vin
- wire segments 35 -> 42
- no-connect marks 4 -> 0
Other:
- note removed: "1"
- note removed: "Holes"
- note removed: "Shield for Arduino Nano"

Commit message: Ctrl unit kicad - separate mcu voltage regulator
Parts:
- added U1: MP2307, converter_dcdc:MP2037, symbol control-unit-pcb:MP2307-1265
- C3, C4: footprint (none) -> Capacitor_SMD:C_1206_3216Metric_Pad1.42x1.75mm_HandSolder
- R8, R9: footprint (none) -> Resistor_SMD:R_1206_3216Metric_Pad1.42x1.75mm_HandSolder
Connections:
- net labels added: +7.5V, +BATT
- wire segments 42 -> 38

Commit message: Update ctrl module schema
Parts:
- R1, R2, R3, R4, R5, R6, R7: footprint (none) -> Resistor_SMD:R_1206_3216Metric_Pad1.42x1.75mm_HandSolder
- U1: symbol control-unit-pcb:MP2307-1265 -> control-unit-pcb-rescue:MP2307-1265-control-unit-pcb
Changed lines of the file:
@@
 F 0 "R3" V 4700 3900 50  0000 C CNN
 F 1 "R" V 4650 3750 50  0000 C CNN
-F 2 "" V 4680 3750 50  0001 C CNN
+F 2 "Resistor_SMD:R_1206_3216Metric_Pad1.42x1.75mm_HandSolder" V 4680 3750 50  0001 C CNN
 F 3 "~" H 4750 3750 50  0001 C CNN
 	1    4750 3750
@@
 F 0 "R4" V 4700 4000 50  0000 C CNN
 F 1 "R" V 4634 3850 50  0000 C CNN
-F 2 "" V 4680 3850 50  0001 C CNN
+F 2 "Resistor_SMD:R_1206_3216Metric_Pad1.42x1.75mm_HandSolder" V 4680 3850 50  0001 C CNN
 F 3 "~" H 4750 3850 50  0001 C CNN
 	1    4750 3850
@@
 F 0 "R5" V 4700 4100 50  0000 C CNN
 F 1 "R" V 4634 3950 50  0000 C CNN
-F 2 "" V 4680 3950 50  0001 C CNN
+F 2 "Resistor_SMD:R_1206_3216Metric_Pad1.42x1.75mm_HandSolder" V 4680 3950 50  0001 C CNN
 F 3 "~" H 4750 3950 50  0001 C CNN
 	1    4750 3950
@@
 F 0 "R6" V 4700 4200 50  0000 C CNN
 F 1 "R" V 4634 4050 50  0000 C CNN
-F 2 "" V 4680 4050 50  0001 C CNN
+F 2 "Resistor_SMD:R_1206_3216Metric_Pad1.42x1.75mm_HandSolder" V 4680 4050 50  0001 C CNN
 F 3 "~" H 4750 4050 50  0001 C CNN
 	1    4750 4050
@@
 F 0 "R2" V 4700 3800 50  0000 C CNN
 F 1 "1k2" V 4700 3950 50  0000 C CNN
-F 2 "" V 4680 3650 50  0001 C CNN
+F 2 "Resistor_SMD:R_1206_3216Metric_Pad1.42x1.75mm_HandSolder" V 4680 3650 50  0001 C CNN
 F 3 "~" H 4750 3650 50  0001 C CNN
 	1    4750 3650
@@
 F 0 "R1" V 4200 3150 50  0000 C CNN
 F 1 "2k2" V 4400 3100 50  0000 C CNN
-F 2 "" V 4230 3150 50  0001 C CNN
+F 2 "Resistor_SMD:R_1206_3216Metric_Pad1.42x1.75mm_HandSolder" V 4230 3150 50  0001 C CNN
 F 3 "~" H 4300 3150 50  0001 C CNN
 	1    4300 3150
@@
 F 0 "R7" H 6730 3754 50  0000 R CNN
 F 1 "R" H 6730 3845 50  0000 R CNN
-F 2 "" V 6730 3800 50  0001 C CNN
+F 2 "Resistor_SMD:R_1206_3216Metric_Pad1.42x1.75mm_HandSolder" V 6730 3800 50  0001 C CNN
 F 3 "~" H 6800 3800 50  0001 C CNN
 	1    6800 3800
@@
 $EndComp
 $Comp
-L control-unit-pcb:MP2307-1265 U1
+L control-unit-pcb-rescue:MP2307-1265-control-unit-pcb U1
 U 1 1 5EE9C12C
 P 6000 2400
